Commit message: docs(readme): update quick-start notes with lerobot-env, STL export, leader-arm teleop
- lerobot-env now built (conda, Python 3.12, LeRobot 0.6.2) and documented,
  including the [dataset] extra and SOCKS-proxy gotchas hit during setup
- note that the official demo dataset + checkpoint are already downloaded
- add scripts/tools/usd_to_stl.py to export assets/props/*.usd to real-scale
  STL for 3D printing, plus the converted files in assets/props_stl/
- document real leader-arm hardware teleop end to end: dialout group
  permission fix, calibration, teleop_agent.py --task vs record_episodes.py
  --env inconsistency, and its 25s default --episode-length causing
  premature resets
- pick up so101_w_cam.urdf's auto-corrected mesh paths (meshes/ -> ../meshes/,
  fixes relative paths from the urdf/ subdirectory) produced when Isaac Sim
  loaded the robot during leader-arm testing

Co-Authored-By: Claude Sonnet 5 <noreply@anthropic.com>

File: assets/robots/so101/urdf/so101_w_cam.urdf (robot description, URDF)
Before this commit: robot so101_w_cam, 9 links, 8 joints
Links:
- link base_link: geometry collision mesh filename=../meshes/base_motor_holder_so101_v1.stl; collision mesh filename=../meshes/base_so101_v2.stl
- link camera_wrist: geometry collision mesh filename=../meshes/camera_box.stl; visual mesh filename=../meshes/camera_box.stl
- link gripper_link: geometry collision mesh filename=../meshes/sts3215_03a_v1.stl; collision mesh filename=../meshes/wrist_roll_follower_so101_w_cam_mount_right.stl
- link lower_arm_link: geometry collision mesh filename=../meshes/motor_holder_so101_wrist_v1.stl; collision mesh filename=../meshes/sts3215_03a_v1.stl
- link moving_jaw_so101_v1_link: geometry collision mesh filename=../meshes/moving_jaw_so101_v1.stl; visual mesh filename=../meshes/moving_jaw_so101_v1.stl
- link shoulder_link: geometry collision mesh filename=../meshes/motor_holder_so101_base_v1.stl; collision mesh filename=../meshes/rotation_pitch_so101_v1.stl
- link upper_arm_link: geometry collision mesh filename=../meshes/sts3215_03a_v1.stl; collision mesh filename=../meshes/upper_arm_so101_v1.stl
- link wrist_link: geometry collision mesh filename=../meshes/sts3215_03a_no_horn_v1.stl; collision mesh filename=../meshes/wrist_roll_pitch_so101_v2.stl
